File: ch340k.kicad_pcb (KiCad board)
At the start: 2 copper layers, 33 x 17.8 mm, 8 parts, among them J1 USB_B_Mini, J2 Conn_01x06_Male, U1 CH340K

Commit message: CW Interface prototype
Parts:
- removed F1: Fuse, digikey-footprints:0603
- added C1: 0.1u, UserLib:0603, F.Cu at (137.9, 79.4)
- added C1: 0.1u, UserLib:0603, B.Cu at (141.0, 72.4)
- added C1: 0.1u, UserLib:0603, B.Cu at (141.0, 80.0)
- added C2: 10u, Capacitor_THT:CP_Radial_D5.0mm_P2.00mm, F.Cu at (138.4, 74.9)
- added C3: 0.1u, UserLib:0603, F.Cu at (134.6, 71.8)
- added C4: 10u, Capacitor_THT:CP_Radial_D5.0mm_P2.00mm, F.Cu at (130.5, 69.8)
- added J3: Conn_01x02_Male, Connector_PinHeader_2.54mm:PinHeader_1x02_P2.54mm_Vertical, F.Cu at (144.8, 78.7)
- added J4: Conn_01x02_Male, Connector_PinHeader_2.54mm:PinHeader_1x02_P2.54mm_Vertical, F.Cu at (144.8, 71.1)
- added R4: 1k, UserLib:0603, B.Cu at (133.3, 69.8)
- added R5: 1k, UserLib:0603, F.Cu at (138.4, 71.1)
- added U2: TLP290, Package_SO:SOP-4_4.4x2.6mm_P1.27mm, B.Cu at (134.6, 81.3)
- added U3: TLP290, Package_SO:SOP-4_4.4x2.6mm_P1.27mm, B.Cu at (134.6, 72.4)
- D1: footprint digikey-footprints:LED_2-SMD_No_Lead_1.7x0.8mm -> UserLib:0603
- J2: value Conn_01x06_Male -> Conn_01x03_Male; footprint Connector_PinHeader_2.54mm:PinHeader_1x06_P2.54mm_Vertical -> Connector_PinHeader_2.54mm:PinHeader_1x03_P2.54mm_Vertical
- R1, R2: value 0 -> 1k; footprint digikey-footprints:0603 -> UserLib:0603; moved to B.Cu
- R3: value 10k -> 1k; footprint digikey-footprints:0603 -> UserLib:0603
- moved D1 16.7 mm to (116.8, 68.6), turned to 0 degrees
- moved R1 14.4 mm to (128.3, 80.0)
- moved R3 11.3 mm to (120.7, 68.6)
- moved R2 6.35 mm to (128.3, 73.7)
- moved U1 3.98 mm to (132.1, 76.1)
- moved J2 2.54 mm to (142.2, 68.6), turned to -90 degrees
Connections:
- J1 pad 1: Net-(F1-Pad2) -> Net-(J1-Pad1)
- J1 pad 4: Net-(J1-Pad4) -> unconnected-(J1-Pad4)
- J2 pad 1: Net-(J2-Pad1) -> GND
- J2 pad 2: Net-(J2-Pad2) -> Net-(R5-Pad2)
- J2 pad 3: Net-(J2-Pad3) -> Net-(R4-Pad2)
- R1 pad 1: Net-(R1-Pad1) -> Net-(U1-Pad6)
- R1 pad 2: Net-(J2-Pad1) -> Net-(R1-Pad2)
- R2 pad 1: Net-(F1-Pad1) -> Net-(U1-Pad4)
- R2 pad 2: Net-(J2-Pad1) -> Net-(R2-Pad2)
- R3 pad 1: Net-(F1-Pad1) -> Net-(C3-Pad1)
- U1 pad 10: Net-(R1-Pad1) -> Net-(C3-Pad1)
- U1 pad 4: Net-(J2-Pad5) -> Net-(U1-Pad4)
- U1 pad 5: Net-(U1-Pad5) -> unconnected-(U1-Pad5)
- U1 pad 6: Net-(J2-Pad4) -> Net-(U1-Pad6)
- U1 pad 7: Net-(F1-Pad1) -> Net-(J1-Pad1)
- U1 pad 8: Net-(J2-Pad2) -> Net-(U1-Pad8)
- U1 pad 9: Net-(J2-Pad3) -> Net-(U1-Pad9)
Routing:
- net Net-(J1-Pad1): track 0.00 -> 31.5 mm
- net Net-(F1-Pad1): track 27.7 -> 0.00 mm
- net GND: track 13.4 -> 32.6 mm
- net Net-(C3-Pad1): track 0.00 -> 18.6 mm
- net Net-(J2-Pad5): track 17.1 -> 0.00 mm
- net Net-(J2-Pad1): track 14.3 -> 0.00 mm
- net Net-(U1-Pad6): track 0.00 -> 9.33 mm, vias 0 -> 1
- net Net-(J2-Pad3): track 8.64 -> 0.00 mm, vias 2 -> 0
- net Net-(J2-Pad2): track 7.92 -> 0.00 mm, vias 1 -> 0
- net Net-(U1-Pad4): track 0.00 -> 7.85 mm, vias 0 -> 1
- net Net-(C5-Pad2): track 0.00 -> 7.76 mm
- net Net-(C5-Pad1): track 0.00 -> 7.71 mm
- net Net-(J2-Pad4): track 7.41 -> 0.00 mm
- net Net-(C6-Pad2): track 0.00 -> 7.24 mm
- net Net-(C6-Pad1): track 0.00 -> 7.24 mm
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Other:
- board text added: "CH340K"
- board text added: "DTR"
- board text added: "JK1MLY 2022.3"
- board text added: "RTS"
- board text added: "T R"
